Commit message: liveshare with chloe and seth

File: assets/urdf/drone.urdf (robot description, URDF)
Before this commit: robot simple_drone, 9 links, 8 joints
Links:
- link base_link: geometry collision cylinder length=0.05 radius=0.15; visual mesh filename=package://assets/models/drone.obj

Commit message: LiveShare

File: assets/urdf/drone.urdf (robot description, URDF)
Before this commit: robot simple_drone, 9 links, 8 joints
Links:
- link base_link: geometry collision box size=0.3 0.3 0.1; visual mesh filename=meshes/drone.obj scale=1 1 1
